File: Multi Programmer.kicad_pcb (KiCad board)
At the start: 2 copper layers, 99.1 x 96.5 mm, 66 parts, among them J1 USB_B, J2 Serial, SW1 RESET, SW2 MODE, U1 TTLSW, U2 FT232RL, U3 ATmega328P-PU, U4 NE555, Y1 16MHz, Y2 16MHz

Commit message: Repositioned crystal
Parts:
- moved Y2 39.3 mm to (146.7, 111.8), turned to 0 degrees
- moved C24 37.6 mm to (147.3, 107.3), turned to 180 degrees
- moved C25 32.6 mm to (151.1, 107.3), turned to 0 degrees
Routing:
- net /S_XTAL1: track 50.8 -> 70.3 mm, vias 0 -> 1
- net /S_XTAL2: track 51.8 -> 67.4 mm, vias 0 -> 1
- net GND: track 615.1 -> 605.6 mm, vias 23 -> 29
- net /S_SCK: track 197.1 -> 193.4 mm
- net Net-(SK2-Pad12): track 7.62 -> 9.09 mm
- net Net-(SK2-Pad11): track 7.62 -> 8.67 mm
- net /S_MOSI: track 186.1 -> 185.5 mm
Other:
- board text added: "SOCKET CRYSTAL"
