File: Multi Programmer.sch (KiCad schematic (older format))
At the start: 64 parts, among them J1 USB_B, J2 Serial, SW1 RESET, SW2 MODE, U1 TTLSW, U2 FT232RL, U3 ATmega328P-PU, U4 NE555, Y1 16MHz, Y2 16MHz

Commit message: Added sockets for attiny, move sockets to separate page
Parts:
- removed C1, C18, C2: 100n, Capacitor_SMD:C_0805_2012Metric_Pad1.15x1.40mm_HandSolder, symbol Device:C_Small
- removed C11, C12: 22p, Capacitor_SMD:C_0805_2012Metric_Pad1.15x1.40mm_HandSolder, symbol Device:C_Small
- removed JP1, JP2: Jumper, Connector_PinHeader_2.54mm:PinHeader_1x02_P2.54mm_Vertical, symbol Device:Jumper
- removed SK1: ATmega328P-AU, Package_DIP:DIP-32_W15.24mm_Socket, symbol MCU_Microchip_ATmega:ATmega328P-AU
- removed SK2: ATmega328P-PU, DTLib:DIP-28_Zif_Multi, symbol MCU_Microchip_ATmega:ATmega328P-PU
- removed Y2: 16MHz, Crystal:Crystal_HC18-U_Vertical, symbol Device:Crystal_Small
Connections:
- net labels removed: S_XTAL1, S_XTAL2
- wire segments 269 -> 228
- no-connect marks 55 -> 23
Other:
- note removed: "PROGRAMMING SOCKETS"
- note removed: "SOCKET CRYSTAL"

Commit message: 
Parts:
- added C1, C11, C12, C18, C2: 100n, Capacitor_SMD:C_0805_2012Metric_Pad1.15x1.40mm_HandSolder, symbol Device:C_Small
- added C24, C25: 22, Capacitor_SMD:C_0805_2012Metric_Pad1.15x1.40mm_HandSolder, symbol Device:C_Small
- added SK1: ATmega328P-AU, Package_DIP:DIP-32_W15.24mm_Socket, symbol MCU_Microchip_ATmega:ATmega328P-AU
- added SK2: ATmega328P-PU, DTLib:DIP-28_Zif_Multi, symbol MCU_Microchip_ATmega:ATmega328P-PU
- added SK3: ATtiny45/85, Package_DIP:DIP-8_W7.62mm, symbol MCU_Microchip_ATtiny:ATtiny85-20PU
- added SK4: ATtiny44/84, Package_DIP:DIP-14_W7.62mm, symbol MCU_Microchip_ATtiny:ATtiny84A-PU
- added Y2: 16MHz, Crystal:Crystal_HC18-U_Vertical, symbol Device:Crystal_Small
- C8, C9: value 100n -> 22
Connections:
- net labels added: S_XTAL1, S_XTAL2
- wire segments 228 -> 287
- no-connect marks 23 -> 65
Other:
- note added: "ATMEGA328p"
- note added: "ATTINY44/84"
- note added: "ATTINY45/85"

Commit message: Repositioned crystal
Other:
- note added: "SOCKETED CRYSTAL"
- moved on the sheet: C10, C11, C12, C13, C14, C15, C16, C17, C20, C21, C22, C23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
